File: titancore-7960_industrial/titancore-7960_industrial.kicad_sch (KiCad schematic)
At the start: 28 parts, among them J1 XT30, J2 Pin Header M 01x08, J3 XT30, J4 XT30, Q1 BTN8982TA, Q2 BTN8982TA, Q3 BTN8982TA, Q4 BTN8982TA, U5 74HC244

Commit message: led
Parts:
- added D1: Red LED, LED_SMD:LED_0805_2012Metric, symbol Device:LED
- added R15: 10k, Resistor_SMD:R_0805_2012Metric_Pad1.20x1.40mm_HandSolder, symbol Device:R_US
Connections:
- net GND: now also R15.2
- net VS: now also D1.2 (A)
- new net: D1.1 (K), R15.1
Changed lines of the file:
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@@
 	)
 	(junction
+		(at 39.37 21.59)
+		(diameter 0)
+		(color 0 0 0 0)
+	)
+	(junction
 		(at 113.03 72.39)
 		(diameter 0)
@@
 	)
 	(junction
+		(at 33.02 29.21)
+		(diameter 0)
+		(color 0 0 0 0)
+	)
+	(junction
 		(at 113.03 102.87)
 		(diameter 0)
@@
 	)
 	(junction
-		(at 39.37 21.59)
+		(at 69.85 46.99)
 		(diameter 0)
 		(color 0 0 0 0)
 	)
 	(junction
-		(at 69.85 46.99)
+		(at 52.07 21.59)
 		(diameter 0)
 		(color 0 0 0 0)
@@
 	(wire
 		(pts
-			(xy 39.37 29.21) (xy 33.02 29.21)
+			(xy 33.02 29.21) (xy 41.91 29.21)
 		)
 		(stroke
@@
 	(wire
 		(pts
-			(xy 45.72 21.59) (xy 39.37 21.59)
-		)
-		(stroke
-			(width 0)
-			(type default)
-		)
-	)
-	(wire
-		(pts
 			(xy 138.43 48.26) (xy 153.67 48.26)
 		)
@@
 	(wire
 		(pts
-			(xy 46.99 29.21) (xy 39.37 29.21)
+			(xy 113.03 52.07) (xy 121.92 52.07)
 		)
 		(stroke
@@
 	(wire
 		(pts
-			(xy 113.03 52.07) (xy 121.92 52.07)
+			(xy 138.43 105.41) (xy 153.67 105.41)
 		)
 		(stroke
@@
 	(wire
 		(pts
-			(xy 138.43 105.41) (xy 153.67 105.41)
+			(xy 118.11 62.23) (xy 138.43 62.23)
 		)
 		(stroke
@@
 	(wire
 		(pts
-			(xy 118.11 62.23) (xy 138.43 62.23)
+			(xy 118.11 33.02) (xy 138.43 33.02)
 		)
 		(stroke
@@
 	(wire
 		(pts
-			(xy 118.11 33.02) (xy 138.43 33.02)
+			(xy 102.87 124.46) (xy 69.85 124.46)
 		)
 		(stroke
@@
 	(wire
 		(pts
-			(xy 102.87 124.46) (xy 69.85 124.46)
+			(xy 52.07 21.59) (xy 39.37 21.59)
 		)
 		(stroke
@@
 	(wire
 		(pts
+			(xy 52.07 21.59) (xy 55.88 21.59)
+		)
+		(stroke
+			(width 0)
+			(type default)
+		)
+	)
+	(wire
+		(pts
 			(xy 123.19 22.86) (xy 123.19 29.21)
 		)
@@
 	(wire
 		(pts
+			(xy 49.53 29.21) (xy 52.07 29.21)
+		)
+		(stroke
+			(width 0)
+			(type default)
+		)
+	)
+	(wire
+		(pts
 			(xy 99.06 127) (xy 102.87 127)
 		)
@@
 	)
 	(symbol
+		(lib_id "Device:R_US")
+		(at 45.72 29.21 270)
+		(unit 1)
+		(body_style 1)
+		(exclude_from_sim no)
+		(in_bom yes)
+		(on_board yes)
+		(in_pos_files yes)
+		(dnp no)
+		(property "Reference" "R15"
+			(at 44.196 31.496 90)
+			(show_name no)
+			(do_not_autoplace no)
+			(effects
+				(font
+					(size 1.27 1.27)
+				)
+				(justify right)
+			)
+		)
+		(property "Value" "10k"
+			(at 50.292 31.496 90)
+			(show_name no)
+			(do_not_autoplace no)
+			(effects
+				(font
+					(size 1.27 1.27)
+				)
+				(justify right)
+			)
+		)
+		(property "Footprint" "Resistor_SMD:R_0805_2012Metric_Pad1.20x1.40mm_HandSolder"
+			(at 45.466 30.226 90)
+			(hide yes)
+			(show_name no)
+			(do_not_autoplace no)
+			(effects
+				(font
+					(size 1.27 1.27)
+				)
+			)
+		)
+		(property "Datasheet" ""
+			(at 45.72 29.21 0)
+			(hide yes)
+			(show_name no)
+			(do_not_autoplace no)
+			(effects
+				(font
+					(size 1.27 1.27)
+				)
+			)
+		)
+		(property "Description" "Resistor, US symbol"
+			(at 45.72 29.21 0)
+			(hide yes)
+			(show_name no)
+			(do_not_autoplace no)
+			(effects
+				(font
+					(size 1.27 1.27)
+				)
+			)
+		)
+		(pin "1"
+		)
+		(pin "2"
+		)
+		(instances
+			(project "titancore-7960_industrial"
+				(path "/742efa3c-2585-473f-9559-a4f38a1ea3b9"
+					(reference "R15")
+					(unit 1)
+				)
+			)
+		)
+	)
+	(symbol
 		(lib_id "power:VS")
 		(at 113.03 52.07 0)
@@
 	(symbol
 		(lib_id "power:VS")
-		(at 45.72 21.59 270)
+		(at 55.88 21.59 270)
 		(unit 1)
 		(body_style 1)
@@
 		(fields_autoplaced yes)
 		(property "Reference" "#PWR03"
-			(at 41.91 21.59 0)
+			(at 52.07 21.59 0)
 			(hide yes)
 			(show_name no)
@@
 		)
 		(property "Value" "VS"
-			(at 49.53 21.5899 90)
+			(at 59.69 21.5899 90)
 			(show_name no)
 			(do_not_autoplace no)
@@
 		)
 		(property "Footprint" ""
-			(at 45.72 21.59 0)
+			(at 55.88 21.59 0)
 			(hide yes)
 			(show_name no)
@@
 		)
 		(property "Datasheet" ""
-			(at 45.72 21.59 0)
+			(at 55.88 21.59 0)
 			(hide yes)
 			(show_name no)
@@
 		)
 		(property "Description" "Power symbol creates a global label with name \"VS\""
-			(at 45.72 21.59 0)
+			(at 55.88 21.59 0)
 			(hide yes)
 			(show_name no)
@@
 	(symbol
 		(lib_id "power:GND")
-		(at 46.99 29.21 0)
+		(at 33.02 29.21 0)
 		(unit 1)
 		(body_style 1)
@@
 		(dnp no)
 		(property "Reference" "#PWR015"
-			(at 46.99 35.56 0)
+			(at 33.02 35.56 0)
 			(hide yes)
 			(show_name no)
@@
 		)
 		(property "Value" "GND"
-			(at 46.99 32.512 0)
+			(at 33.02 32.512 0)
 			(show_name no)
 			(do_not_autoplace no)
@@
 		)
 		(property "Footprint" ""
-			(at 46.99 29.21 0)
+			(at 33.02 29.21 0)
 			(hide yes)
 			(show_name no)
@@
 		)
 		(property "Datasheet" ""
-			(at 46.99 29.21 0)
+			(at 33.02 29.21 0)
 			(hide yes)
 			(show_name no)
@@
 		)
 		(property "Description" "Power symbol creates a global label with name \"GND\" , ground"
-			(at 46.99 29.21 0)
+			(at 33.02 29.21 0)
 			(hide yes)
 			(show_name no)
@@
 					(unit 1)
 				)
+			)
+		)
+	)
+	(symbol
+		(lib_id "Device:LED")
+		(at 52.07 25.4 90)
+		(unit 1)
+		(body_style 1)
+		(exclude_from_sim no)
+		(in_bom yes)
+		(on_board yes)
+		(in_pos_files yes)
+		(dnp no)
+		(property "Reference" "D1"
+			(at 55.88 26.67 90)
+			(show_name no)
+			(do_not_autoplace no)
+			(effects
+				(font
+					(size 1.27 1.27)
+				)
+			)
+		)
+		(property "Value" "Red LED"
+			(at 57.404 24.892 90)
+			(show_name no)
+			(do_not_autoplace no)
+			(effects
+				(font
+					(size 1.27 1.27)
+				)
+			)
+		)
+		(property "Footprint" "LED_SMD:LED_0805_2012Metric"
+			(at 52.07 25.4 0)
+			(hide yes)
+			(show_name no)
+			(do_not_autoplace no)
+			(effects
+				(font
+					(size 1.27 1.27)
+				)
+			)
+		)
+		(property "Datasheet" ""
+			(at 52.07 25.4 0)
+			(hide yes)
+			(show_name no)
+			(do_not_autoplace no)
+			(effects
+				(font
+					(size 1.27 1.27)
+				)
+			)
+		)
+		(property "Description" "Light emitting diode"
+			(at 52.07 25.4 0)
+			(hide yes)
+			(show_name no)
+			(do_not_autoplace no)
+			(effects
+				(font
+					(size 1.27 1.27)
+				)
+			)
+		)
+		(property "Sim.Pins" "1=K 2=A"
+			(at 52.07 25.4 0)
+			(hide yes)
+			(show_name no)
+			(do_not_autoplace no)
+			(effects
+				(font
+					(size 1.27 1.27)
+				)
+			)
+		)
+		(pin "1"
+		)
+		(pin "2"
+		)
+		(instances
+			(project "titancore-7960_industrial"
+				(path "/742efa3c-2585-473f-9559-a4f38a1ea3b9"
+					(reference "D1")
+					(unit 1)
+				)
